File: AUTOCROFT MVP VERSION 1.0/Autocroft Node PCB ver2/Autocroft_node/Autocroft_node.kicad_pcb (KiCad board)
At the start: 2 copper layers, 77 x 55 mm, 18 parts, among them J1 MOISTURE-SENSOR, J2 DS3231, J3 HC-12, J4 BLUEPILL, Q1 IRLZ44N, U1 L7805, U2 LM358, U3 EEPROM

Commit message: Node PCB
Parts:
- added  : MountingHole_2.2mm_M2, MountingHole:MountingHole_2.2mm_M2, F.Cu at (140.4, 91.5)
- added  : MountingHole_2.2mm_M2, MountingHole:MountingHole_2.2mm_M2, F.Cu at (197.2, 44.9)
- J3: footprint Connector_PinSocket_2.54mm:PinSocket_1x04_P2.54mm_Vertical -> Connector_PinSocket_2.54mm:PinSocket_1x05_P2.54mm_Vertical
Connections:
- J4 pad 33: Net-(J4-Pad33) -> PB0
Routing:
- net PB0: track 0.00 -> 34.9 mm
- net GND: track 227.3 -> 229.1 mm, vias 0 -> 5
- net VCC_5V: vias 0 -> 1
- added copper zone on B.Cu, net GND
- added copper zone on F.Cu, net GND
Other:
- board text added: "+"
- board text added: "-"
