File: AUTOCROFT MVP VERSION 1.0/Node PCB Ver1/Autocroft_node/Autocroft_node.kicad_pcb (KiCad board)
At the start: 2 copper layers, 77 x 55 mm, 20 parts, among them J1 MOISTURE-SENSOR, J2 DS3231, J3 HC-12, J4 BLUEPILL, Q1 IRLZ44N, U1 L7805, U2 LM358, U3 EEPROM

Commit message: update
Other:
- net class Default removed
- net class Power removed
